File: rs70.sch (KiCad schematic (older format))
At the start: 30 parts, among them U1 ATSAMS70J21B-MN

Commit message: test
Parts:
- removed C? (x7): 100nF, symbol Device:C
- added C10, C11, C13, C14, C15, C16, C9: 100nF, symbol Device:C_Small
- C1, C12, C3, C4, C5, C6, C7, C8: renamed from C?; symbol Device:C -> Device:C_Small
- L1: renamed from L?; value 10μH - 60mA -> 10μH-60mA; symbol pspice:INDUCTOR -> Device:L_Small
- L2: renamed from L?; symbol pspice:INDUCTOR -> Device:L_Small
- R1, R2, R5: renamed from R?; symbol Device:R -> Device:R_Small
- gave numbers to parts that had none: 9
Connections:
- wire segments 83 -> 89
- no-connect marks 4 -> 9
Other:
- moved on the sheet: C1, C12, C3, C4, C5, C6, C7, C8, R1, R2, R5, U1B
